File: CueOMatic.kicad_pcb (KiCad board)
At the start: 2 copper layers, 30.2 x 52.5 mm, 9 parts, among them J1 TTL, J3 POGO_IN, J4 POGO_OUT, SW4 SW_DIP_x04, U2 UA78M33_TO252, U3 esp-01m

Commit message: Pre milling
Parts:
- added SW2: MODE, pts636:pts636, F.Cu at (106.4, 67.2)
- added SW3: RESET, pts636:pts636, F.Cu at (112.8, 92.5)
- moved J1 1.36 mm to (103.1, 80.8)
- moved J3 0.64 mm to (102.8, 97.4)
- moved J4 0.64 mm to (126.5, 97.4)
- moved U3 0.57 mm to (111.5, 75.5)
Connections:
- U3 pad 7: Net-(U3-GP2) -> unconnected-(U3-GP2-Pad7)
Routing:
- net I2C_SDA: track 47.9 -> 58.6 mm
- net I2C_SCL: track 46.8 -> 56.9 mm
- net +3V3: track 82.6 -> 91.1 mm
- net GND: track 6.26 -> 14.3 mm
- net VBUS: track 78.5 -> 84.8 mm
- net Net-(U3-GP0): track 0.00 -> 4.30 mm
- net Net-(U3-RST): track 0.00 -> 4.14 mm
- net unconnected-(U3-GP13-Pad5): track 0.00 -> 2.57 mm, vias 0 -> 1
- net unconnected-(U3-GP4-Pad10): track 0.00 -> 2.08 mm, vias 0 -> 1
- net RX: track 6.21 -> 7.50 mm
- net TX: track 5.82 -> 6.78 mm
